File: oso-o-46.kicad_sch (KiCad schematic)
At the start: 137 parts

Commit message: Capacitor capacitance was incorrect.
Parts:
- C1, C2: LCSC C1729 -> (none)
- C3: value (none) -> 1u; footprint (none) -> Capacitor_SMD:C_0805_2012Metric_Pad1.18x1.45mm_HandSolder
- C4, C5, C6: value (none) -> 0.1u; footprint (none) -> Capacitor_SMD:C_0603_1608Metric_Pad1.08x0.95mm_HandSolder
- C7: value (none) -> 10u; footprint (none) -> Capacitor_SMD:C_0805_2012Metric_Pad1.18x1.45mm_HandSolder
- D1: value (none) -> LED; footprint (none) -> LED_SMD:LED_0603_1608Metric_Pad1.05x0.95mm_HandSolder
- D10, D11, D12, D13, D14, D15, D16, D17, D18, D19, D2, D20, D21, D22, D23, D24, D25, D26, D27, D28, D29, D3, D30, D31, D32, D33, D34, D35, D36, D37, D38, D39, D4, D40, D41, D42, D43, D44, D45, D46, D47, D48, D49, D5, D50, D51, D52, D53, D54, D55, D56, D57, D58, D59, D6, D7, D8, D9: value (none) -> D; footprint (none) -> Diode_SMD:D_SOD-123
- F1: value (none) -> ASMD1206-150; footprint (none) -> Fuse:Fuse_1206_3216Metric_Pad1.42x1.75mm_HandSolder
- R1, R7: value (none) -> 10k; footprint (none) -> Resistor_SMD:R_0805_2012Metric
- R2, R5: value (none) -> 5.1k; footprint (none) -> Resistor_SMD:R_0805_2012Metric
- R3, R4: value (none) -> 22; footprint (none) -> Resistor_SMD:R_0805_2012Metric
- R6: value (none) -> 1k; footprint (none) -> Resistor_SMD:R_0805_2012Metric
- SW1: value (none) -> SW_Push; footprint (none) -> Button_Switch_SMD:SW_SPST_B3U-1000P
- SW10, SW11, SW12, SW13, SW14, SW15, SW16, SW17, SW18, SW19, SW2, SW20, SW21, SW22, SW23, SW24, SW25, SW26, SW27, SW28, SW29, SW3, SW30, SW31, SW32, SW33, SW34, SW35, SW36, SW37, SW38, SW39, SW4, SW40, SW41, SW42, SW43, SW44, SW45, SW46, SW47, SW48, SW49, SW5, SW50, SW51, SW52, SW53, SW54, SW55, SW56, SW57, SW58, SW59, SW6, SW7, SW8, SW9: value (none) -> SW_PUSH; footprint (none) -> Switch_Keyboard_Kailh:SW_Kailh_Choc_V1
- U1: value (none) -> PRTR5V0U2X; footprint (none) -> Package_TO_SOT_SMD:SOT-143
- U2: value (none) -> ATmega32U4-A; footprint (none) -> Package_QFP:TQFP-44_10x10mm_P0.8mm
- USB1: value (none) -> HRO-TYPE-C-31-M-12; footprint (none) -> Type-C:HRO-TYPE-C-31-M-12-Assembly
- Y1: value (none) -> 16HMz; footprint (none) -> Crystal:Crystal_SMD_3225-4Pin_3.2x2.5mm_HandSoldering
